File: Etch_A_Tune/Etch_A_Tune.kicad_sch (KiCad schematic)
At the start: 5 parts, among them J1 UJ20-C-H-G-MSMT-2-P16-TR, J2 TSM-117-01-F-DV-P-TR, J3 TSM-115-01-T-DV-P-TR, J4 TSM-110-01-T-DV-P, J5 TSM-108-01-L-DV-A-P-TR

Commit message: Updated schematic and preliminary PCB doc
did rough PCB layout
Parts:
- added S6: 450404015514, 450404015514, symbol SamacSys_Parts:450404015514
Other:
- moved on the sheet: J1, J2, J3, J4, J5

Commit message: Schematic Update
Fixed component Footprints and added new switches/rotary encoders. Wired and placed bypass capacitors for most devices. Removed 5V boost converter because external DAC is no longer being utilized. Placed uC onto board design and implemented charging through USB-C connector.
Parts:
- removed J1: UJ20-C-H-G-MSMT-2-P16-TR, UJ20CHGMSMT2P16TR, symbol SamacSys_Parts:UJ20-C-H-G-MSMT-2-P16-TR
- removed J2: TSM-117-01-F-DV-P-TR, TSM-117-YY-ZZZ-DV-P-TR, symbol SamacSys_Parts:TSM-117-01-F-DV-P-TR
- removed J3: TSM-115-01-T-DV-P-TR, TSM-115-YY-ZZZ-DV-P-TR, symbol SamacSys_Parts:TSM-115-01-T-DV-P-TR
- removed J4: TSM-110-01-T-DV-P, TSM-110-YY-ZZZ-DV-P, symbol SamacSys_Parts:TSM-110-01-T-DV-P
- removed J5: TSM-108-01-L-DV-A-P-TR, TSM-108-YY-ZZZ-DV-A-P-TR, symbol SamacSys_Parts:TSM-108-01-L-DV-A-P-TR
- removed S6: 450404015514, 450404015514, symbol SamacSys_Parts:450404015514
- added J2: 2171790001, BQ25170DSGR:MOLEX_2171790001, symbol 2171790001:2171790001
- added TP1, TP4: TestPoint, TestPoint:TestPoint_Pad_D1.0mm, symbol Connector:TestPoint
Connections:
- new net Battery/USB_Power: J2.A4B9 (VBUS1), J2.B4A9 (VBUS2), TP1.1
- new net GND: J2.A1B12 (GND1), J2.B1A12 (GND2), TP4.1
- no-connect marks 0 -> 12
Other:
- removed sheet DAC
- added sheet Microcontroller (Microcontroller.kicad_sch)
- sheet Battery ports: added BAT_DIAG, PG, USB_Power; removed Charge
- sheet Controllers ports: added ROTA1, ROTA2, ROTB1, ROTB2, ROTP1, ROTP2, SlideSwitch; removed ROT1, ROT2
- sheet Power ports: added Power; removed 3.3V, 5v

Commit message: Etch A Tune V.02
Updated more foot prints and components onto bom, specifically SWD debug header and 1x14 pin header for touch and screen module. Added 4pin header for SD card reader.
Parts:
- added J1: RSM-114-02-T-S, BQ25170DSGR:SAMTEC_RSM-114-02-T-S, symbol RSM-114-02-T-S:RSM-114-02-T-S
- added J2: 91601-304ALF, BQ25170DSGR:AMPHENOL_91601-304ALF, symbol 91601-304ALF:91601-304ALF
- added J3: M20-7910542R, BQ25170DSGR:HARWIN_M20-7910542R, symbol M20-7910542R:M20-7910542R
- renumbered J2 to J4, TP4 to TP1, TP1 to TP2
Connections:
- net GND: now also J1.13, J3.5
- new net +3.3V: J1.14
- new net CS: J1.12
- new net DC/RS: J1.10
- new net LED: J1.07
- new net RESET: J1.11
- new net SCK: J1.08
- new net SDI (MOSI): J1.09
- new net SDO(MISO): J1.06
- new net SD_CS: J2.01
- new net SD_MISO: J2.03
- new net SD_MOSI: J2.02
- new net SD_SCK: J2.04
- new net SWCLK: J3.3
- new net SWDIO: J3.2
- new net SWO: J3.4
- new net SWRESET: J3.1
- new net T_CLK: J1.05
- new net T_CS: J1.04
- new net T_DIN: J1.03
- new net T_DO: J1.02
- new net T_IRQ: J1.01
Other:
- sheet Microcontroller ports: added SCREEN_BACKLIGHT, SCREEN_DCRS, SCREEN_MISO, SCREEN_MOSI, SCREEN_RESET, SCREEN_SCK, SCREEN_SS, SD_MISO, SD_MOSI, SD_SCK, SD_SS, SWCLK, SWDIO, SWO, SWRESET, TOUCH_IRQ, TOUCH_MISO, TOUCH_MOSI, TOUCH_SCK, TOUCH_SS; removed SPI5_MISO, SPI5_MOSI, SPI5_SCK, SPI5_SS

Commit message: Updated parallel power supply
Updated USB and battery operation and added DAC output
Parts:
- added J5: SJ-3524-SMT-PI, BQ25170DSGR:CUI_SJ-3524-SMT-PI, symbol SJ-3524-SMT-PI:SJ-3524-SMT-PI
- added TP16, TP17, TP18, TP19, TP20, TP21, TP22, TP23, TP24, TP25, TP26, TP27, TP28, TP29, TP30, TP31, TP32, TP33, TP34, TP35: TestPoint, TestPoint:TestPoint_Pad_D1.0mm, symbol Connector:TestPoint
Connections:
- net CS: now also TP16.1
- net DC/RS: now also TP18.1
- net LED: now also TP21.1
- net RESET: now also TP17.1
- net SCK: now also TP20.1
- net SDI (MOSI): now also TP19.1
- net SDO(MISO): now also TP22.1
- net SD_CS: now also TP28.1
- net SD_MISO: now also TP30.1
- net SD_MOSI: now also TP29.1
- net SD_SCK: now also TP31.1
- net SWCLK: now also TP34.1
- net SWDIO: now also TP33.1
- net SWO: now also TP35.1
- net SWRESET: now also TP32.1
- net T_CLK: now also TP23.1
- net T_CS: now also TP24.1
- net T_DIN: now also TP25.1
- net T_DO: now also TP26.1
- net T_IRQ: now also TP27.1
Other:
- sheet Battery ports: added BAT_V_SENSE, PACK+; removed Power
- sheet Microcontroller ports: added BAT_V_SENSE, DAC_OUT; removed none
- sheet Power ports: added PACK+, USB_Power; removed Power

Commit message: V.04 Schematic
added 64 pin header LEDS
Parts:
- added J6: 6130XX243121_613064243121, 6130XX243121_613064243121:613064243121, symbol 6130XX243121_613064243121:6130XX243121_613064243121
Other:
- moved on the sheet: J1, J2, TP16, TP17, TP18, TP19, TP20, TP21, TP22, TP23, TP24, TP25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

Commit message: Updated schematic
Parts:
- removed J3: M20-7910542R, BQ25170DSGR:HARWIN_M20-7910542R, symbol M20-7910542R:M20-7910542R
- removed TP35: TestPoint, TestPoint:TestPoint_Pad_D1.0mm, symbol Connector:TestPoint
- added J7: 3220-10-0300-00, 3220-10-0300-00:CNC_3220-10-0300-00, symbol 3220-10-0300-00:3220-10-0300-00
- added TP39: TestPoint, TestPoint:TestPoint_Pad_D1.0mm, symbol Connector:TestPoint
Connections:
- net SWRESET is gone; now on net SWDIO: TP32.1
- net +3.3V: now also J7.1
- net GND: now also J7.3, J7.5, J7.9
- net SWCLK: now also TP33.1, J7.4; no longer TP34.1
- net SWDIO: now also J7.2; no longer TP33.1
- net SWO: now also TP34.1, J7.6
- new net nRESET: J7.10, TP39.1
- no-connect marks 12 -> 14
Other:
- moved on the sheet: TP32, TP33, TP34

Commit message: Final Layout before routing
Parts:
- removed J1: RSM-114-02-T-S, BQ25170DSGR:SAMTEC_RSM-114-02-T-S, symbol RSM-114-02-T-S:RSM-114-02-T-S
- added C8: 330uF, Capacitor_SMD:C_0603_1608Metric, symbol Device:C
- added J1: 75915-414LF, BQ25170DSGR:75915414LF, symbol 75915-414LF:75915-414LF
- added R22, R23: 5.1k, Resistor_SMD:R_0603_1608Metric, symbol Device:R
- added R24, R25: 0, Resistor_SMD:R_0603_1608Metric, symbol Device:R
- J6: footprint 6130XX243121_613064243121:613064243121 -> BQ25170DSGR:613064243121
- J7: footprint 3220-10-0300-00:CNC_3220-10-0300-00 -> BQ25170DSGR:CNC_3220-10-0300-00
Connections:
- net +3.3V: now also J1.14
- net CS: now also J1.12
- net DC/RS: now also J1.10
- net GND: now also J5.1, J1.13, R22.2, R23.2
- net LED: now also J1.7
- net Microcontroller/DAC_OUT: now also C8.1
- net RESET: now also J1.11
- net SCK: now also J1.8
- net SDI (MOSI): now also J1.9
- net SDO(MISO): now also J1.6
- net T_CLK: now also J1.5
- net T_CS: now also J1.4
- net T_DIN: now also J1.3
- net T_DO: now also J1.2
- net T_IRQ: now also J1.1
- net PE3: now reaches J6.1
- net PD13: now reaches J6.10
- net PF6: now reaches J6.11
- net PD14: now reaches J6.12
- net PF7: now reaches J6.13
- net PD15: now reaches J6.14
- net PF8: now reaches J6.15
- net PG6: now reaches J6.16
- net PF9: now reaches J6.17
- net PG7: now reaches J6.18
- net PF10: now reaches J6.19
- net PD9: now reaches J6.2
- net PG8: now reaches J6.20
- net PC0: now reaches J6.21
- net PC6: now reaches J6.22
- net PC1: now reaches J6.23
- net PC7: now reaches J6.24
- net PC2_C: now reaches J6.25
- net PC8: now reaches J6.26
- net PC3_C: now reaches J6.27
- net PC9: now reaches J6.28
- net PB11: now reaches J6.29
- net PE4: now reaches J6.3
- net PA8: now reaches J6.30
- net PB10: now reaches J6.31
- net PA9: now reaches J6.32
- net PE15: now reaches J6.33
- net PA10: now reaches J6.34
- net PE14: now reaches J6.35
- net PA11: now reaches J6.36
- net PE13: now reaches J6.37
- net PA12: now reaches J6.38
- net PE12: now reaches J6.39
- net PD10: now reaches J6.4
- net PE1: now reaches J6.40
- net PE11: now reaches J6.41
- net PE0: now reaches J6.42
- net PE10: now reaches J6.43
- net PB9: now reaches J6.44
- net PE9: now reaches J6.45
- net PB8: now reaches J6.46
- net PE8: now reaches J6.47
- net PB7: now reaches J6.48
- net PE7: now reaches J6.49
- net PE5: now reaches J6.5
- net PB6: now reaches J6.50
- net PF15: now reaches J6.51
- net PB5: now reaches J6.52
- net PF14: now reaches J6.53
- net PB4: now reaches J6.54
- net PF11: now reaches J6.55
- net PB2: now reaches J6.57
- net PA2: now reaches J6.59
- net PD11: now reaches J6.6
- net PA1: now reaches J6.61
- net PA0: now reaches J6.63
- net PE6: now reaches J6.7
- net PD12: now reaches J6.8
- net PC13: now reaches J6.9
- net at J4.A5 (CC1): now also R23.1
- net at J4.B5 (CC2): now also R22.1
- net at J5.2: now also R25.2
- net at J5.3: now also R24.2
- new net: C8.2, R24.1, R25.1
- no-connect marks 14 -> 18
Other:
- moved on the sheet: J2, J4, J5, J6, J7, TP1, TP16, TP17, TP18, TP19, TP2, TP20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

Commit message: Update
Connections:
- net +3.3V: now also J6.56, J6.58
- net GND: now also J4.SH1 (SHIELD1), J4.SH2 (SHIELD2), J4.SH3 (SHIELD3), J4.SH4 (SHIELD4), J6.62, J6.64
- net Battery/USB_Power renamed Battery/USB_Charge
- no-connect marks 18 -> 10
Other:
- sheet Battery ports: added USB_Charge; removed USB_Power
