File: Etch_A_Tune/Etch_A_Tune.kicad_sch (KiCad schematic)
At the start: 33 parts, among them J1 75915-414LF, J2 91601-304ALF, J4 2171790001, J5 SJ-3524-SMT-PI, J6 6130XX243121_613064243121, J7 3220-10-0300-00

Commit message: Another Update! :D
Parts:
- removed J6: 6130XX243121_613064243121, BQ25170DSGR:613064243121, symbol 6130XX243121_613064243121:6130XX243121_613064243121
- renumbered C8 to C1, J4 to J1, J7 to J3, J1 to J4, R23 to R1, R22 to R2, R24 to R3, R25 to R4, TP39 to TP10, TP16 to TP11, TP17 to TP12, TP18 to TP13, TP19 to TP14, TP20 to TP15, TP21 to TP16, TP22 to TP17, TP23 to TP18, TP24 to TP19, TP25 to TP20, TP26 to TP21, TP27 to TP22, TP28 to TP3, TP29 to TP4, TP30 to TP5, TP31 to TP6, TP32 to TP7, TP33 to TP8, TP34 to TP9
Connections:
- no-connect marks 10 -> 9

Commit message: pdf docs
Parts:
- renumbered C1 to C8, J4 to J1, J1 to J4, J3 to J7, R2 to R22, R1 to R23, R3 to R24, R4 to R25, TP11 to TP16, TP12 to TP17, TP13 to TP18, TP14 to TP19, TP15 to TP20, TP16 to TP21, TP17 to TP22, TP18 to TP23, TP19 to TP24, TP20 to TP25, TP21 to TP26, TP22 to TP27, TP3 to TP28, TP4 to TP29, TP5 to TP30, TP6 to TP31, TP7 to TP32, TP8 to TP33, TP9 to TP34, TP10 to TP39

Commit message: 95% finished PCB
Only changes needed for completion is ferrite bead footprint and DNP crystal osc.
Parts:
- added J3, J6: 91601-304ALF, BQ25170DSGR:AMPHENOL_91601-304ALF, symbol 91601-304ALF:91601-304ALF
Connections:
- new net PA0: J3.04
- new net PA1: J3.03
- new net PA10: J6.03
- new net PA11: J6.04
- new net PA2: J3.02
- new net PA8: J6.01
- new net PA9: J6.02
- new net PC1: J3.01
Other:
- sheet Microcontroller ports: added PA0, PA1, PA10, PA11, PA2, PA8, PA9, PC1; removed none

Commit message: Update
Changed DC blocking cap to 1206 footprint, added SVG silkscreen to back of board and added team name date and version
Parts:
- C8: footprint Capacitor_SMD:C_0603_1608Metric -> Capacitor_SMD:C_1210_3225Metric
Changed lines of the file:
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@@
 			)
 		)
-		(property "Footprint" "Capacitor_SMD:C_0603_1608Metric"
+		(property "Footprint" "Capacitor_SMD:C_1210_3225Metric"
 			(at 346.71 214.9348 0)
 			(effects

Commit message: Updated BOM
Changed Values for an accurate BOM, and exported results
Parts:
- C8: DIGIKEY-PURCHASE-URL (none) -> https://www.digikey.com/short/jfp3nd05; Dist (none) -> Digikey; Dist Part Number (none) -> 4713-GMC32X5R337M6R3NTCT-ND; Manufacturer_Name (none) -> Cal-Chip Electronics, Inc.; Manufacturer_Part_Number (none) -> GMC32X5R337M6R3NT; Price (none) -> $4.26
- J1: DIGIKEY-PURCHASE-URL (none) -> https://www.digikey.com/short/m553pr9w; Dist (none) -> Digikey; Dist Part Number (none) -> 609-75915-414LF-ND; Price (none) -> $1.86
- J2, J3, J6: DIGIKEY-PURCHASE-URL (none) -> https://www.digikey.com/short/th748djz; Dist (none) -> Digikey; Dist Part Number (none) -> 609-91601-304ALFCT-ND; Manufacturer_Name (none) -> Amphenol ICC (FCI); Manufacturer_Part_Number (none) -> 91601-304ALF; Price (none) -> $0.76
- J4: DIGIKEY-PURCHASE-URL (none) -> https://www.digikey.com/short/99h5mzt5; Dist (none) -> Digikey; Dist Part Number (none) -> 900-2171790001CT-ND; Manufacturer_Name (none) -> Molex; Manufacturer_Part_Number (none) -> 2171790001; Price (none) -> $0.83
- J5: DIGIKEY-PURCHASE-URL (none) -> https://www.digikey.com/short/t4tqnp4v; Dist (none) -> Digikey; Dist Part Number (none) -> CP-3524SJPICT-ND; Manufacturer_Name (none) -> Same Sky (Formerly CUI Devices); Manufacturer_Part_Number (none) -> SJ-3524-SMT-TR-PI; Price (none) -> $1.22
- J7: DIGIKEY-PURCHASE-URL (none) -> https://www.digikey.com/short/nh549v4d; Dist (none) -> Digikey; Dist Part Number (none) -> 1175-1629-ND; Manufacturer_Name (none) -> CNC Tech; Manufacturer_Part_Number (none) -> 3220-10-0300-00; Price (none) -> $0.81
- R22, R23: DIGIKEY-PURCHASE-URL (none) -> https://www.digikey.com/short/2dq5m4th; Dist (none) -> Digikey; Dist Part Number (none) -> 311-5.1KGRCT-ND; Manufacturer_Name (none) -> YAGEO; Manufacturer_Part_Number (none) -> RC0603JR-075K1L; Price (none) -> $0.10
- R24, R25: DIGIKEY-PURCHASE-URL (none) -> https://www.digikey.com/short/7nbcpfpb; Dist (none) -> Digikey; Dist Part Number (none) -> 311-0.0GRCT-ND; Manufacturer_Name (none) -> YAGEO; Manufacturer_Part_Number (none) -> RC0603JR-070RL; Price (none) -> $0.10
- TP1, TP16, TP17, TP18, TP19, TP2, TP20, TP21, TP22, TP23, TP24, TP25, TP26, TP27, TP28, TP29, TP30, TP31, TP32, TP33, TP34, TP39: Dist (none) -> Digikey; now left out of the parts list
