File: Etch_A_Tune/Microcontroller.kicad_sch (KiCad schematic)
At the start: 4 parts, among them U4 STM32H7A3ZIT6Q

Commit message: Etch A Tune V.02
Updated more foot prints and components onto bom, specifically SWD debug header and 1x14 pin header for touch and screen module. Added 4pin header for SD card reader.
Parts:
- renumbered C1 to C6, C11 to C7, R32 to R19, U4 to U5
Connections:
- net BAT_DIAG: no longer U5.134 (PB7)
- net ROTA1: no longer U5.111 (PC12)
- net ROTA2: no longer U5.114 (PD2)
- net ROTB1: no longer U5.110 (PC11)
- net ROTB2: no longer U5.113 (PD1)
- net ROTP1: no longer U5.109 (PC10)
- net ROTP2: no longer U5.112 (PD0)
- net SW1: no longer U5.115 (PD3)
- net SW2: no longer U5.116 (PD4)
- net SW3: no longer U5.117 (PD5)
- net SW4: no longer U5.120 (PD6)
- net SW5: no longer U5.121 (PD7)
- net SWRESET: now also U5.27 (NRST)
- net SlideSwitch: no longer U5.133 (PB6)
- net SCREEN_SS: now reaches U5.43 (PA4)
- net SCREEN_SCK: now reaches U5.44 (PA5)
- net SCREEN_MOSI: now reaches U5.45 (PA6)
- net SCREEN_MISO: now reaches U5.46 (PA7)
- net SCREEN_RESET: now reaches U5.47 (PC4)
- net SCREEN_DCRS: now reaches U5.48 (PC5)
- net SCREEN_BACKLIGHT: now reaches U5.49 (PB0)
- net TOUCH_SS: now reaches U5.72 (PB12)
- net SD_SS: now reaches U5.108 (PA15)
- net TOUCH_SCK: now reaches U5.73 (PB13)
- net TOUCH_MOSI: now reaches U5.74 (PB14)
- net TOUCH_MISO: now reaches U5.75 (PB15)
- net TOUCH_IRQ: now reaches U5.76 (PD8)
- new net SD_MISO: U5.111 (PC12)
- new net SD_MOSI: U5.110 (PC11)
- new net SD_SCK: U5.109 (PC10)
Other:
- moved on the sheet: C7, R19

Commit message: Updated parallel power supply
Updated USB and battery operation and added DAC output
Connections:
- net BAT_DIAG: now also U5.126 (PG13)
- net GND: now also U5.118 (VSS)
- net PG: now also U5.127 (PG14)
- net ROTA1: now also U5.114 (PD2)
- net ROTA2: now also U5.117 (PD5)
- net ROTB1: now also U5.113 (PD1)
- net ROTB2: now also U5.116 (PD4)
- net ROTP1: now also U5.112 (PD0)
- net ROTP2: now also U5.115 (PD3)
- net SCREEN_BACKLIGHT: now also U5.50 (PB1); no longer U5.49 (PB0)
- net SCREEN_DCRS: now also U5.49 (PB0); no longer U5.48 (PC5)
- net SCREEN_RESET: now also U5.48 (PC5); no longer U5.47 (PC4)
- net SCREEN_SS: now also U5.47 (PC4); no longer U5.43 (PA4)
- net SW1: now also U5.120 (PD6)
- net SW2: now also U5.121 (PD7)
- net SW3: now also U5.122 (PG9)
- net SW4: now also U5.123 (PG10)
- net SW5: now also U5.124 (PG11)
- net SlideSwitch: now also U5.125 (PG12)
- net BAT_V_SENSE: now reaches U5.40 (PA3)
- new net DAC_OUT: U5.43 (PA4)

Commit message: V.04 Schematic
added 64 pin header LEDS
Parts:
- added D2: 150060GS75000, symbol Device:LED
- added R21: R, symbol Device:R
Connections:
- net GND: now also D2.1 (K)
- net at U5.1 (PE2): now also R21.1
- new net: D2.2 (A), R21.2

Commit message: Updated schematic
Connections:
- net PE3: now reaches U5.2 (PE3)
- net PF6: now reaches U5.20 (PF6)
- net PF7: now reaches U5.21 (PF7)
- net PF8: now reaches U5.22 (PF8)
- net PF9: now reaches U5.23 (PF9)
- net PF10: now reaches U5.24 (PF10)
- net PC0: now reaches U5.28 (PC0)
- net PC1: now reaches U5.29 (PC1)
- net PE4: now reaches U5.3 (PE4)
- net PC2_C: now reaches U5.30 (PC2_C)
- net PC3_C: now reaches U5.31 (PC3_C)
- net PE5: now reaches U5.4 (PE5)
- net PE6: now reaches U5.5 (PE6)
- net PE11: now reaches U5.61 (PE11)
- net PE12: now reaches U5.62 (PE12)
- net PE13: now reaches U5.63 (PE13)
- net PE14: now reaches U5.64 (PE14)
- net PE15: now reaches U5.65 (PE15)
- net PB10: now reaches U5.66 (PB10)
- net PB11: now reaches U5.67 (PB11)
- net PC13: now reaches U5.9 (PC13)
Other:
- moved on the sheet: D2, R21

Commit message: Final Layout before routing
Parts:
- removed C7: 100n, oresat-passives:0603-C-NOSILK, symbol Device:C_Small
- removed R19: 10k, oresat-passives:0603-C-NOSILK, symbol Device:R_Small_US
- added R19: 10k, Resistor_SMD:R_0603_1608Metric, symbol Device:R
- C6: value C -> 100nF; footprint (none) -> Capacitor_SMD:C_0603_1608Metric
- D2: footprint (none) -> LED_SMD:LED_0603_1608Metric
- R21: value R -> 10; footprint (none) -> Resistor_SMD:R_0603_1608Metric
Connections:
- net GND is gone; now on net +3.3V: C6.2, D2.1 (K), U5.118 (VSS), U5.12 (VSS), U5.18 (VSS), U5.33 (VSS), U5.34 (VSSA), U5.41 (VSS), U5.55 (VSS), U5.6 (VSS), U5.69 (VSS)
- net +3.3V: now also R19.1; no longer C6.1
- net SWCLK: now also U5.107 (PA14)
- net SWDIO: now also U5.102 (PA13)
- net SWO: now also U5.130 (PB3)
- net SWRESET: now also C6.1, R19.2
- net PA0: now reaches U5.37 (PA0)
- net PA1: now reaches U5.38 (PA1)
- net PA2: now reaches U5.39 (PA2)
- net PB2: now reaches U5.51 (PB2)
- net PF11: now reaches U5.52 (PF11)
- net PF14: now reaches U5.53 (PF14)
- net PF15: now reaches U5.54 (PF15)
- net PE7: now reaches U5.57 (PE7)
- net PE8: now reaches U5.58 (PE8)
- net PE9: now reaches U5.59 (PE9)
- net PE10: now reaches U5.60 (PE10)
- net PA11: now reaches U5.100 (PA11)
- net PA12: now reaches U5.101 (PA12)
- net PB4: now reaches U5.131 (PB4)
- net PB5: now reaches U5.132 (PB5)
- net PB6: now reaches U5.133 (PB6)
- net PB7: now reaches U5.134 (PB7)
- net PB8: now reaches U5.136 (PB8)
- net PB9: now reaches U5.137 (PB9)
- net PE0: now reaches U5.138 (PE0)
- net PE1: now reaches U5.139 (PE1)
- net PD9: now reaches U5.77 (PD9)
- net PD10: now reaches U5.78 (PD10)
- net PD11: now reaches U5.81 (PD11)
- net PD12: now reaches U5.82 (PD12)
- net PD13: now reaches U5.83 (PD13)
- net PD14: now reaches U5.84 (PD14)
- net PD15: now reaches U5.85 (PD15)
- net PG6: now reaches U5.86 (PG6)
- net PG7: now reaches U5.87 (PG7)
- net PG8: now reaches U5.88 (PG8)
- net PC6: now reaches U5.93 (PC6)
- net PC7: now reaches U5.94 (PC7)
- net PC8: now reaches U5.95 (PC8)
- net PC9: now reaches U5.96 (PC9)
- net PA8: now reaches U5.97 (PA8)
- net PA9: now reaches U5.98 (PA9)
- net PA10: now reaches U5.99 (PA10)

Commit message: Update
Parts:
- removed C6: 100nF, Capacitor_SMD:C_0603_1608Metric, symbol Device:C
Connections:
- net +3.3V: no longer D2.1 (K), U5.118 (VSS), U5.12 (VSS), U5.13 (VDD), U5.18 (VSS), U5.19 (VDD), U5.32 (VDD), U5.33 (VSS), U5.34 (VSSA), U5.36 (VDDA), U5.41 (VSS), U5.55 (VSS), U5.6 (VSS), U5.69 (VSS), U5.7 (VDD), U5.8 (VBAT)
- now unconnected: U5.42 (VDD), U5.56 (VDD), U5.71 (VDD)
- no-connect marks 9 -> 49

Commit message: Another Update! :D
Parts:
- removed R19: 10k, Resistor_SMD:R_0603_1608Metric, symbol Device:R
- added C10, C11, C14, C19, C20, C21, C22, C23, C26, C27, C28, C29, C30, C32, C33, C34, C35, C8, C9: 100nF, symbol Device:C
- added C12, C18: 100n, oresat-passives:0603-C-NOSILK, symbol Device:C_Small
- added C13, C31: 1uF, symbol Device:C
- added C15: 220pF, symbol Device:C
- added C16, C17: 1u, oresat-passives:0603-C-NOSILK, symbol Device:C_Small
- added C24, C25: 18pf, symbol Device:C
- added C36: 4.7uF, symbol Device:C
- added FB1: FerriteBead_Small, symbol Device:FerriteBead_Small
- added R38: 10k, Resistor_SMD:R_0603_1608Metric, symbol Device:R
- added R39, R40: 0, Resistor_SMD:R_0603_1608Metric, symbol Device:R
- added TP39: USB5V, TestPoint:TestPoint_Pad_D1.0mm, symbol Connector:TestPoint
- added TP40: USB3V3, TestPoint:TestPoint_Pad_D1.0mm, symbol Connector:TestPoint
- added TP41: BOOT0, TestPoint:TestPoint_Pad_D1.0mm, symbol Connector:TestPoint
- added Y1: 12Mhz, Crystal:Crystal_SMD_Abracon_ABM8G-4Pin_3.2x2.5mm, symbol Device:Crystal_GND24
- renumbered R21 to R37, U5 to U6
Connections:
- net +3.3V: now also U6.105 (VDDLDO), U6.106 (VDD), U6.119 (VDDMMC), U6.129 (VDD), U6.13 (VDD), U6.143 (VDDLDO), U6.144 (VDD), U6.19 (VDD), U6.32 (VDD), U6.56 (VDD), U6.70 (VDDLDO), U6.71 (VDD), U6.79 (VDD), U6.8 (VBAT), U6.92 (VDD), C10.1, C11.1, C13.1, C14.1, C19.1, C21.1, C22.1, C23.1, C31.1, C33.1, C34.1, C35.1, C36.1, C8.1, C9.1, FB1.2, R38.1, R39.2
- net SWRESET: now also C12.1, R38.2
- net GND: now reaches U6.12 (VSS)
- net GND: now also U6.104 (VSS), U6.118 (VSS), U6.128 (VSS), U6.14 (VSSSMPS), U6.141 (VSS), U6.17 (VFBSMPS), U6.18 (VSS), U6.33 (VSS), U6.34 (VSSA), U6.41 (VSS), U6.55 (VSS), U6.6 (VSS), U6.69 (VSS), U6.80 (VSS), U6.89 (VSS), C12.2, C15.2, C19.2, C20.1, C21.2, C22.2, C23.2, C24.2, C25.2, C29.1, C31.2, C32.1, C33.2, C34.2, C35.2, C36.2, R40.2, Y1.2, Y1.4
- net at U6.15 (VLXSMPS): now also C15.1
- net at U6.35 (VREF+): now also C16.1
- net at U6.36 (VDDA): now also C17.1, C18.1, FB1.1
- net VCORE: now reaches U6.68 (VCAP)
- net VCORE: now also U6.140 (VCAP), C20.2, C29.2, C32.2
- net at U6.135 (BOOT0): now also TP41.1
- net at U6.142 (PDR_ON): now also R39.1, R40.1
- net at U6.90 (VDD50USB): now also TP39.1
- net at U6.91 (VDD33USB): now also TP40.1
- net PA10: no longer names the net of U6.99 (PA10)
- net PA11: no longer names the net of U6.100 (PA11)
- net PA12: no longer names the net of U6.101 (PA12)
- net PA8: no longer names the net of U6.97 (PA8)
- net PA9: no longer names the net of U6.98 (PA9)
- net PB10: no longer names the net of U6.66 (PB10)
- net PB11: no longer names the net of U6.67 (PB11)
- net PB2: no longer names the net of U6.51 (PB2)
- net PB4: no longer names the net of U6.131 (PB4)
- net PB5: no longer names the net of U6.132 (PB5)
- net PB6: no longer names the net of U6.133 (PB6)
- net PB7: no longer names the net of U6.134 (PB7)
- net PB8: no longer names the net of U6.136 (PB8)
- net PB9: no longer names the net of U6.137 (PB9)
- net PC0: no longer names the net of U6.28 (PC0)
- net PC1: no longer names the net of U6.29 (PC1)
- net PC2_C: no longer names the net of U6.30 (PC2_C)
- net PC3_C: no longer names the net of U6.31 (PC3_C)
- net PC6: no longer names the net of U6.93 (PC6)
- net PC7: no longer names the net of U6.94 (PC7)
- net PC8: no longer names the net of U6.95 (PC8)
- net PC9: no longer names the net of U6.96 (PC9)
- net PD10: no longer names the net of U6.78 (PD10)
- net PD11: no longer names the net of U6.81 (PD11)
- net PD12: no longer names the net of U6.82 (PD12)
- net PD13: no longer names the net of U6.83 (PD13)
- net PD14: no longer names the net of U6.84 (PD14)
- net PD15: no longer names the net of U6.85 (PD15)
- net PD9: no longer names the net of U6.77 (PD9)
- net PE0: no longer names the net of U6.138 (PE0)
- net PE1: no longer names the net of U6.139 (PE1)
- net PE10: no longer names the net of U6.60 (PE10)
- net PE11: no longer names the net of U6.61 (PE11)
- net PE12: no longer names the net of U6.62 (PE12)
- net PE13: no longer names the net of U6.63 (PE13)
- net PE14: no longer names the net of U6.64 (PE14)
- net PE15: no longer names the net of U6.65 (PE15)
- net PE3: no longer names the net of U6.2 (PE3)
- net PE4: no longer names the net of U6.3 (PE4)
- net PE5: no longer names the net of U6.4 (PE5)
- net PE6: no longer names the net of U6.5 (PE6)
- net PE7: no longer names the net of U6.57 (PE7)
- net PE8: no longer names the net of U6.58 (PE8)
- net PE9: no longer names the net of U6.59 (PE9)
- net PF10: no longer names the net of U6.24 (PF10)
- net PF11: no longer names the net of U6.52 (PF11)
- net PF14: no longer names the net of U6.53 (PF14)
- net PF15: no longer names the net of U6.54 (PF15)
- net PF6: no longer names the net of U6.20 (PF6)
- net PF7: no longer names the net of U6.21 (PF7)
- net PF8: no longer names the net of U6.22 (PF8)
- net PF9: no longer names the net of U6.23 (PF9)
- net PG6: no longer names the net of U6.86 (PG6)
- net PG7: no longer names the net of U6.87 (PG7)
- net PG8: no longer names the net of U6.88 (PG8)
- new net: C10.2, C11.2, C13.2, C14.2, C16.2, C17.2, C18.2, C8.2, C9.2
- new net: C26.1, C27.1, C28.1, C30.1
- new net: C26.2, C27.2, C28.2, C30.2
- new net OSC_H_IN: C24.1, Y1.1
- new net OSC_H_OUT: C25.1, Y1.3
- no-connect marks 49 -> 65
Other:
- note added: "Crystal Oscillator"
- note added: "Place Each Near A Different VDD"
- note added: "Place Each Near A Different VDD and VDDLDO"
- note added: "Place Near VBatt Pin"
- note added: "Place Near VCAP"
- note added: "Place Near VCCMMC"
- note added: "Place Near VDDA Pin"
- moved on the sheet: D2, R37, U6A

Commit message: pdf docs
Parts:
- renumbered C11 to C10, C14 to C11, C13 to C12, C19 to C13, C21 to C14, C22 to C15, C20 to C16, C32 to C17, C29 to C18, C23 to C19, C30 to C20, C28 to C21, C27 to C22, C26 to C23, C33 to C24, C31 to C25, C34 to C26, C36 to C27, C35 to C28, C15 to C32, C17 to C33, C18 to C34, C16 to C35, C24 to C36, C25 to C37, C8 to C6, C10 to C6, C12 to C7, C9 to C7, R39 to R19, R37 to R21, R38 to R39, TP39 to TP35, U6 to U5, Y1 to Y2
