File: Etch_A_Tune/Microcontroller.kicad_sch (KiCad schematic)
At the start: 40 parts, among them U5 STM32H7A3ZIT6Q, Y2 12Mhz

Commit message: PCB about 75% done
Parts:
- removed C10, C11, C13, C14, C15, C16, C17, C18, C19, C20, C21, C22, C23, C24, C26, C28, C6 (x2), C7: 100nF, symbol Device:C
- removed C12, C25: 1uF, symbol Device:C
- removed C27: 4.7uF, symbol Device:C
- removed C32: 220pF, symbol Device:C
- removed C33, C35: 1u, oresat-passives:0603-C-NOSILK, symbol Device:C_Small
- removed C34, C7: 100n, oresat-passives:0603-C-NOSILK, symbol Device:C_Small
- removed C36, C37: 18pf, symbol Device:C
- removed FB1: FerriteBead_Small, symbol Device:FerriteBead_Small
- removed R39: 10k, Resistor_SMD:R_0603_1608Metric, symbol Device:R
- removed R40: 0, Resistor_SMD:R_0603_1608Metric, symbol Device:R
- removed TP35: USB5V, TestPoint:TestPoint_Pad_D1.0mm, symbol Connector:TestPoint
- removed TP40: USB3V3, TestPoint:TestPoint_Pad_D1.0mm, symbol Connector:TestPoint
- removed TP41: BOOT0, TestPoint:TestPoint_Pad_D1.0mm, symbol Connector:TestPoint
- removed Y2: 12Mhz, Crystal:Crystal_SMD_Abracon_ABM8G-4Pin_3.2x2.5mm, symbol Device:Crystal_GND24
- R19: value 0 -> 10k
Connections:
- net +3.3V: now also R19.1; no longer R19.2, U5.105 (VDDLDO), U5.106 (VDD), U5.119 (VDDMMC), U5.129 (VDD), U5.13 (VDD), U5.143 (VDDLDO), U5.144 (VDD), U5.19 (VDD), U5.32 (VDD), U5.56 (VDD), U5.70 (VDDLDO), U5.71 (VDD), U5.79 (VDD), U5.8 (VBAT), U5.92 (VDD)
- net GND: now also D2.1 (K); no longer U5.104 (VSS), U5.118 (VSS), U5.12 (VSS), U5.128 (VSS), U5.14 (VSSSMPS), U5.141 (VSS), U5.17 (VFBSMPS), U5.18 (VSS), U5.33 (VSS), U5.34 (VSSA), U5.41 (VSS), U5.55 (VSS), U5.6 (VSS), U5.69 (VSS), U5.80 (VSS), U5.89 (VSS)
- net SWRESET: now also R19.2
- net at U5.142 (PDR_ON): no longer R19.1
- net VCORE: no longer names the net of U5.68 (VCAP)
- net VCORE: no longer U5.140 (VCAP)
- no-connect marks 65 -> 103
Other:
- note removed: "Crystal Oscillator"
- note removed: "Place Each Near A Different VDD"
- note removed: "Place Each Near A Different VDD and VDDLDO"
- note removed: "Place Near VBatt Pin"
- note removed: "Place Near VCAP"
- note removed: "Place Near VCCMMC"
- note removed: "Place Near VDDA Pin"

Commit message: Update
Finished Analog Power Domain
Parts:
- added C10, C11, C13, C14, C15, C16, C17, C18, C19, C20, C21, C22, C23, C24, C26, C28, C29, C6, C7: 100nF, Capacitor_SMD:C_0603_1608Metric, symbol Device:C
- added C12, C25, C30, C31: 1uF, Capacitor_SMD:C_0603_1608Metric, symbol Device:C
- added C27: 4.7uF, Capacitor_SMD:C_0603_1608Metric, symbol Device:C
- added C32: 220pF, Capacitor_SMD:C_0603_1608Metric, symbol Device:C
- added C33: 1nF, Capacitor_SMD:C_0603_1608Metric, symbol Device:C
- added FB1: FerriteBead_Small, symbol Device:FerriteBead_Small
- added R39, R40: 0, Resistor_SMD:R_0603_1608Metric, symbol Device:R
- added TP35: USB5V, TestPoint:TestPoint_Pad_D1.0mm, symbol Connector:TestPoint
- added TP40: USB3V3, TestPoint:TestPoint_Pad_D1.0mm, symbol Connector:TestPoint
- added TP41: BOOT0, TestPoint:TestPoint_Pad_D1.0mm, symbol Connector:TestPoint
Connections:
- net +3.3V: now also U5.105 (VDDLDO), U5.106 (VDD), U5.119 (VDDMMC), U5.129 (VDD), U5.13 (VDD), U5.143 (VDDLDO), U5.144 (VDD), U5.19 (VDD), U5.32 (VDD), U5.42 (VDD), U5.56 (VDD), U5.7 (VDD), U5.70 (VDDLDO), U5.71 (VDD), U5.79 (VDD), U5.8 (VBAT), U5.92 (VDD), C10.1, C11.1, C12.1, C13.1, C14.1, C15.1, C17.1, C19.1, C20.1, C21.1, C22.1, C23.1, C24.1, C25.1, C26.1, C27.1, C28.1, C6.1, C7.1, FB1.2, R39.2
- net GND: now also U5.104 (VSS), U5.118 (VSS), U5.12 (VSS), U5.128 (VSS), U5.14 (VSSSMPS), U5.141 (VSS), U5.16 (VDDSMPS), U5.17 (VFBSMPS), U5.18 (VSS), U5.33 (VSS), U5.34 (VSSA), U5.41 (VSS), U5.55 (VSS), U5.6 (VSS), U5.69 (VSS), U5.80 (VSS), U5.89 (VSS), C10.2, C11.2, C12.2, C13.2, C14.2, C15.2, C16.1, C17.2, C18.1, C19.2, C20.2, C21.2, C22.2, C23.2, C24.2, C25.2, C26.2, C27.2, C28.2, C29.1, C30.2, C31.2, C32.2, C33.2, C6.2, C7.2, R40.2
- net at U5.15 (VLXSMPS): now also C32.1
- net at U5.35 (VREF+): now also C30.1
- net at U5.36 (VDDA): now also C31.1, C33.1, FB1.1
- net VCORE: now reaches U5.68 (VCAP)
- net VCORE: now also U5.103 (VCAP), U5.140 (VCAP), C16.2, C18.2, C29.2
- net at U5.135 (BOOT0): now also TP41.1
- net at U5.142 (PDR_ON): now also R39.1, R40.1
- net at U5.90 (VDD50USB): now also TP35.1
- net at U5.91 (VDD33USB): now also TP40.1
- net PA0: no longer names the net of U5.37 (PA0)
- net PA1: no longer names the net of U5.38 (PA1)
- net PA2: no longer names the net of U5.39 (PA2)
- net PC13: no longer names the net of U5.9 (PC13)
- no-connect marks 103 -> 63
Other:
- note added: "Place Each Near A Different VDD"
- note added: "Place Each Near A Different VDD and VDDLDO"
- note added: "Place Near VBatt Pin"
- note added: "Place Near VCAP"
- note added: "Place Near VCCMMC"

Commit message: 95% finished PCB
Only changes needed for completion is ferrite bead footprint and DNP crystal osc.
Connections:
- net PC1: now reaches U5.29 (PC1)
- net PA0: now reaches U5.37 (PA0)
- net PA1: now reaches U5.38 (PA1)
- net PA2: now reaches U5.39 (PA2)
- net PA11: now reaches U5.100 (PA11)
- net PA8: now reaches U5.97 (PA8)
- net PA9: now reaches U5.98 (PA9)
- net PA10: now reaches U5.99 (PA10)
- no-connect marks 63 -> 55

Commit message: Finished PCB
Added ferrite bead and crystal oscillator. Added silkscreen text and tidied up component designators.
Parts:
- added C36, C37: 18pf, Capacitor_SMD:C_0603_1608Metric, symbol Device:C
- added Y2: 12Mhz, Crystal:Crystal_SMD_Abracon_ABM8G-4Pin_3.2x2.5mm, symbol Device:Crystal_GND24
- FB1: footprint (none) -> Capacitor_SMD:C_0603_1608Metric
Connections:
- net GND: now also C36.2, C37.2, Y2.2, Y2.4
- net OSC_H_IN: now reaches U5.25 (PH0-OSC_IN)
- net OSC_H_IN: now also C36.1, Y2.1
- net OSC_H_OUT: now reaches U5.26 (PH1-OSC_OUT)
- net OSC_H_OUT: now also C37.1, Y2.3
- no-connect marks 55 -> 53
Other:
- note added: "Crystal Oscillator"

Commit message: Updated BOM
Changed Values for an accurate BOM, and exported results
Parts:
- C10, C11, C13, C14, C15, C16, C17, C18, C19, C20, C21, C22, C23, C24, C26, C28, C29, C6, C7: DIGIKEY-PURCHASE-URL (none) -> https://www.digikey.com/en/products/detail/samsung-electro-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; Dist (none) -> Digikey; Dist Part Number (none) -> 1276-CL10E104KC8VPNCCT-ND; Manufacturer_Name (none) -> Samsung Electro-Mechanics; Manufacturer_Part_Number (none) -> CL10E104KC8VPNC; Price (none) -> $0.25
- C12, C25, C30, C31: DIGIKEY-PURCHASE-URL (none) -> https://www.digikey.com/en/products/detail/samsung-electro-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; Dist (none) -> Digikey; Dist Part Number (none) -> 1276-1184-1-ND; Manufacturer_Name (none) -> Samsung Electro-Mechanics; Manufacturer_Part_Number (none) -> CL10B105KA8NNNC; Price (none) -> $0.08
- C27: DIGIKEY-PURCHASE-URL (none) -> https://www.digikey.com/short/qdh04m32; Dist (none) -> Digikey; Dist Part Number (none) -> 1276-1784-1-ND; Manufacturer_Name (none) -> Samsung Electro-Mechanics; Manufacturer_Part_Number (none) -> CL10A475KO8NNNC; Price (none) -> $0.08
- C32: DIGIKEY-PURCHASE-URL (none) -> https://www.digikey.com/short/727f93v4; Dist (none) -> Digikey; Dist Part Number (none) -> 399-C0603C221K5RACTUCT-ND; Manufacturer_Name (none) -> KEMET; Manufacturer_Part_Number (none) -> C0603C221K5RACTU; Price (none) -> $0.10
- C33: DIGIKEY-PURCHASE-URL (none) -> https://www.digikey.com/short/58b57h08; Dist (none) -> Digikey; Dist Part Number (none) -> 399-C0603C102J8HACAUTOCT-ND; Manufacturer_Name (none) -> KEMET; Manufacturer_Part_Number (none) -> C0603C102J8HACAUTO; Price (none) -> $0.13
- C36, C37: DIGIKEY-PURCHASE-URL (none) -> https://www.digikey.com/short/dz19b2f3; Dist (none) -> Digikey; Dist Part Number (none) -> 399-8828-1-ND; Manufacturer_Name (none) -> KEMET; Manufacturer_Part_Number (none) -> CBR04C180F5GAC; Price (none) -> $0.35
- D2: DIGIKEY-PURCHASE-URL (none) -> https://www.digikey.com/short/5fhtpmbc; Dist (none) -> Digikey; Dist Part Number (none) -> 732-4971-1-ND; Manufacturer_Name (none) -> Würth Elektronik; Manufacturer_Part_Number (none) -> 150060GS75000; Price (none) -> $0.15
- FB1: DIGIKEY-PURCHASE-URL (none) -> https://www.digikey.com/short/t540h2j3; Dist (none) -> Digikey; Dist Part Number (none) -> 490-1014-1-ND; Manufacturer_Name (none) -> Murata Electronics; Manufacturer_Part_Number (none) -> BLM18AG601SN1D; Price (none) -> $0.10
- R19: DIGIKEY-PURCHASE-URL (none) -> https://www.digikey.com/short/m3dw570p; Dist (none) -> Digikey; Dist Part Number (none) -> 311-10.0KHRCT-ND; Manufacturer_Name (none) -> YAGEO; Manufacturer_Part_Number (none) -> RC0603FR-0710KL; Price (none) -> $0.10
- R21: DIGIKEY-PURCHASE-URL (none) -> https://www.digikey.com/short/frnqvwj0; Dist (none) -> Digikey; Dist Part Number (none) -> RMCF0603FT10R0CT-ND; Manufacturer_Name (none) -> Stackpole Electronics Inc; Manufacturer_Part_Number (none) -> RMCF0603FT10R0; Price (none) -> $0.10
- R39: DIGIKEY-PURCHASE-URL (none) -> https://www.digikey.com/short/7nbcpfpb; Dist (none) -> Digikey; Dist Part Number (none) -> 311-0.0GRCT-ND; Manufacturer_Name (none) -> YAGEO; Manufacturer_Part_Number (none) -> RC0603JR-070RL; Price (none) -> $0.10
- R40: DIGIKEY-PURCHASE-URL (none) -> https://www.digikey.com/short/7nbcpfpb; Dist (none) -> Digikey; Dist Part Number (none) -> 311-0.0GRCT-ND; Manufacturer_Name (none) -> YAGEO; Manufacturer_Part_Number (none) -> RC0603JR-070RL; Price (none) -> $0.10; now not fitted
- TP35, TP40, TP41: Dist (none) -> Digikey; now left out of the parts list
- U5: DIGIKEY-PURCHASE-URL (none) -> https://www.digikey.com/short/rrbz14qp; Dist (none) -> Digikey; Dist Part Number (none) -> 497-STM32H7A3ZIT6Q-ND; Manufacturer_Name (none) -> STMicroelectronics; Manufacturer_Part_Number (none) -> STM32H7A3ZIT6Q; Price (none) -> $14.86
- Y2: DIGIKEY-PURCHASE-URL (none) -> https://www.digikey.com/short/j7q5q7v1; Dist (none) -> Digikey; Dist Part Number (none) -> 535-ABM8G-12.000MHZ-D2Y-TCT-ND; Manufacturer_Name (none) -> Abracon LLC; Manufacturer_Part_Number (none) -> ABM8G-12.000MHZ-D2Y-T; Price (none) -> $0.57
