File: Etch_A_Tune/Power.kicad_sch (KiCad schematic)
At the start: 17 parts, among them U4 TPS62063DSGR

Commit message: Updated BOM
Changed Values for an accurate BOM, and exported results
Parts:
- C4, C9: DIGIKEY-PURCHASE-URL (none) -> https://www.digikey.com/short/z7wt55z4; Dist (none) -> Digikey; Dist Part Number (none) -> 1276-1192-1-ND; Manufacturer_Name (none) -> Samsung Electro-Mechanics; Manufacturer_Part_Number (none) -> CL10A106KP8NNNC; Price (none) -> $0.08
- C5: DIGIKEY-PURCHASE-URL (none) -> https://www.digikey.com/short/dmn2thqr; Dist (none) -> Digikey; Dist Part Number (none) -> 399-C0603C220J5GACTUCT-ND; Manufacturer_Name (none) -> KEMET; Manufacturer_Part_Number (none) -> C0603C220J5GACTU; Price (none) -> $0.12
- CR1, CR2: DIGIKEY-PURCHASE-URL (none) -> https://www.digikey.com/short/0t5zd0jr; Dist (none) -> Digikey; Dist Part Number (none) -> CMS06QMCT-ND; Manufacturer_Name (none) -> Toshiba Semiconductor and Storage; Manufacturer_Part_Number (none) -> CMS06(TE12L,Q,M); Price (none) -> $0.23
- D1: DIGIKEY-PURCHASE-URL (none) -> https://www.digikey.com/short/5fhtpmbc; Dist (none) -> Digikey; Dist Part Number (none) -> 732-4971-1-ND; Manufacturer_Name (none) -> Würth Elektronik; Manufacturer_Part_Number (none) -> 150060GS75000; Price (none) -> $0.15
- L1: DIGIKEY-PURCHASE-URL (none) -> https://www.digikey.com/short/hb59fqww; Dist (none) -> Digikey; Dist Part Number (none) -> 587-2164-1-ND; Manufacturer_Name (none) -> Taiyo Yuden; Manufacturer_Part_Number (none) -> BRL3225T1R0M; Price (none) -> $0.18
- R20: DIGIKEY-PURCHASE-URL (none) -> https://www.digikey.com/short/frnqvwj0; Dist (none) -> Digikey; Dist Part Number (none) -> RMCF0603FT10R0CT-ND; Manufacturer_Name (none) -> Stackpole Electronics Inc; Manufacturer_Part_Number (none) -> RMCF0603FT10R0; Price (none) -> $0.10
- R27, R29, R30: DIGIKEY-PURCHASE-URL (none) -> https://www.digikey.com/short/7nbcpfpb; Dist (none) -> Digikey; Dist Part Number (none) -> 311-0.0GRCT-ND; Manufacturer_Name (none) -> YAGEO; Manufacturer_Part_Number (none) -> RC0603JR-070RL; Price (none) -> $0.10
- R5: DIGIKEY-PURCHASE-URL (none) -> https://www.digikey.com/short/8br9tf9h; Dist (none) -> Digikey; Dist Part Number (none) -> P360KHCT-ND; Manufacturer_Name (none) -> Panasonic Electronic Components; Manufacturer_Part_Number (none) -> ERJ-3EKF3603V; Price (none) -> $0.10
- R6: DIGIKEY-PURCHASE-URL (none) -> https://www.digikey.com/short/8797wjjb; Dist (none) -> Digikey; Dist Part Number (none) -> 311-180KGRCT-ND; Manufacturer_Name (none) -> YAGEO; Manufacturer_Part_Number (none) -> RC0603JR-07180KL; Price (none) -> $0.10
- TP36, TP37, TP38: Dist (none) -> Digikey; now left out of the parts list
- U4: DIGIKEY-PURCHASE-URL (none) -> https://www.digikey.com/short/j3qdpjvd; Dist (none) -> Digikey; Dist Part Number (none) -> 296-38304-1-ND; Manufacturer_Name (none) -> Texas Instruments; Manufacturer_Part_Number (none) -> TPS62063DSGR; Price (none) -> $2.12
