File: Etch_A_Tune/Etch_A_Tune.kicad_pcb (KiCad board)
At the start: 4 copper layers, 114.5 x 99.7 mm, 102 parts, among them IC1 BQ25170DSGR, J1 75915-414LF, J2 91601-304ALF, J4 2171790001, J5 SJ-3524-SMT-PI, J6 6130XX243121_613064243121, J7 3220-10-0300-00, U1 BQ297xy, U2 CSD16406Q3, U3 CSD16406Q3, U4 TPS62063DSGR, U5 STM32H7A3ZIT6Q

Commit message: Update
Parts:
- removed C6: 100nF, Capacitor_SMD:C_0603_1608Metric
- removed IC1: BQ25170DSGR, BQ25170DSGR:SON50P200X200X80-9N
- added R31: 10k, Resistor_SMD:R_0603_1608Metric, F.Cu at (196.2, 62.7)
- added R32: 0, Resistor_SMD:R_0603_1608Metric, F.Cu at (196.2, 65.2)
- added R33: 0, Resistor_SMD:R_0603_1608Metric, F.Cu at (196.2, 67.7)
- added R34: 0, Resistor_SMD:R_0603_1608Metric, F.Cu at (196.2, 70.2)
- added R35: 0, Resistor_SMD:R_0603_1608Metric, F.Cu at (196.2, 72.7)
- added R36: 0, Resistor_SMD:R_0603_1608Metric, F.Cu at (196.2, 75.2)
- added R37: 0, Resistor_SMD:R_0603_1608Metric, F.Cu at (196.2, 77.7)
- added R38: 0, Resistor_SMD:R_0603_1608Metric, F.Cu at (196.2, 80.2)
- added U6: BQ25170DSGR, BQ25170DSGR:SON50P200X200X80-9N, F.Cu at (155.6, 30.5)
- R1: value 24k -> 27k
- moved TP23 193.7 mm to (25.5, 73.7)
- moved TP19 191.9 mm to (28.0, 55.2)
- moved TP26 188.1 mm to (28.5, 80.2)
- moved TP18 187.6 mm to (29.0, 57.7)
- moved TP17 183.9 mm to (29.5, 60.2)
- moved TP20 183.2 mm to (27.5, 52.7)
- moved TP16 181.7 mm to (28.5, 62.7)
- moved TP21 181.6 mm to (32.0, 54.7)
- moved TP22 180.0 mm to (36.5, 56.7)
- moved TP25 178.3 mm to (35.0, 75.7)
- moved TP24 176.0 mm to (34.5, 52.7)
- moved R22 162.3 mm to (25.5, 25.7), turned to -90 degrees
- moved S6 124.3 mm to (19.0, 86.2), turned to 90 degrees
- moved TP6 102.6 mm to (126.5, 38.2)
- moved J7 81.0 mm to (103.5, 89.2)
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Connections:
- net /Battery/USB_POWER renamed /Battery/USB_Charge
- C1 pad 2: +3.3V -> GND
- C2 pad 2: +3.3V -> GND
- C4 pad 2: +3.3V -> GND
- C9 pad 2: +3.3V -> GND
- D1 pad 1: +3.3V -> GND
- D2 pad 1: +3.3V -> unconnected-(D2-K-Pad1)
- J1 pad 13: +3.3V -> GND
- J4 pad A1B12: +3.3V -> GND
- J4 pad B1A12: +3.3V -> GND
- J4 pad SH1: unconnected-(J4-SHIELD1-PadSH1) -> GND
- J4 pad SH2: unconnected-(J4-SHIELD2-PadSH2) -> GND
- J4 pad SH3: unconnected-(J4-SHIELD3-PadSH3) -> GND
- J4 pad SH4: unconnected-(J4-SHIELD4-PadSH4) -> GND
- J5 pad 1: +3.3V -> GND
- J6 pad 56: unconnected-(J6-Pad56) -> +3.3V
- J6 pad 58: unconnected-(J6-Pad58) -> +3.3V
- J6 pad 62: unconnected-(J6-Pad62) -> GND
- J6 pad 64: unconnected-(J6-Pad64) -> GND
- J7 pad 3: +3.3V -> GND
- J7 pad 5: +3.3V -> GND
- J7 pad 9: +3.3V -> GND
- MT1 pad C: +3.3V -> GND
- MT1 pad D: +3.3V -> GND
- MT2 pad C: +3.3V -> GND
- MT2 pad D: +3.3V -> GND
- R1 pad 2: +3.3V -> GND
- R2 pad 2: +3.3V -> GND
- R22 pad 2: +3.3V -> GND
- R23 pad 2: +3.3V -> GND
- R4 pad 2: +3.3V -> GND
- R6 pad 2: +3.3V -> GND
- S1 pad 2: +3.3V -> GND
- S2 pad 2: +3.3V -> GND
- S3 pad 2: +3.3V -> GND
- S4 pad 2: +3.3V -> GND
- S5 pad 2: +3.3V -> GND
- S6 pad 3: +3.3V -> GND
- TP1 pad 1: +3.3V -> GND
- U2 pad 4: /Battery/DISCHARGE_GATE -> Net-(R34-Pad2)
- U3 pad 1: +3.3V -> GND
- U3 pad 2: +3.3V -> GND
- U3 pad 3: +3.3V -> GND
- U3 pad 4: /Battery/CHARGE_GATE -> Net-(R33-Pad1)
- U4 pad 1: +3.3V -> GND
- U4 pad 3: +3.3V -> GND
- U4 pad 6: +3.3V -> GND
- U4 pad 9: +3.3V -> GND
- U5 pad 118: +3.3V -> unconnected-(U5B-VSS-Pad118)
- U5 pad 12: +3.3V -> unconnected-(U5A-VSS-Pad12)
- U5 pad 13: +3.3V -> unconnected-(U5A-VDD-Pad13)
- U5 pad 18: +3.3V -> unconnected-(U5A-VSS-Pad18)
- U5 pad 19: +3.3V -> unconnected-(U5A-VDD-Pad19)
- U5 pad 32: +3.3V -> unconnected-(U5A-VDD-Pad32)
- U5 pad 33: +3.3V -> unconnected-(U5A-VSS-Pad33)
- U5 pad 34: +3.3V -> unconnected-(U5A-VSSA-Pad34)
- U5 pad 36: +3.3V -> unconnected-(U5A-VDDA-Pad36)
- U5 pad 41: +3.3V -> unconnected-(U5A-VSS-Pad41)
- U5 pad 42: Net-(U5A-VDD-Pad42) -> unconnected-(U5A-VDD-Pad42)
- U5 pad 55: +3.3V -> unconnected-(U5A-VSS-Pad55)
- U5 pad 56: Net-(U5A-VDD-Pad42) -> unconnected-(U5A-VDD-Pad56)
- U5 pad 6: +3.3V -> unconnected-(U5A-VSS-Pad6)
- U5 pad 69: +3.3V -> unconnected-(U5A-VSS-Pad69)
- U5 pad 7: +3.3V -> unconnected-(U5A-VDD-Pad7)
- U5 pad 71: Net-(U5A-VDD-Pad42) -> unconnected-(U5A-VDD-Pad71)
- U5 pad 8: +3.3V -> unconnected-(U5A-VBAT-Pad8)
Routing:
- net /T_DO: track 0.00 -> 91.0 mm
- net /T_IRQ: track 0.00 -> 86.5 mm, vias 0 -> 1
- net /T_DIN: track 0.00 -> 84.3 mm
- net /T_CLK: track 0.00 -> 75.5 mm, vias 0 -> 2
- net /SD_SCK: track 0.00 -> 67.3 mm
- net /SD_CS: track 0.00 -> 63.4 mm
- net /T_CS: track 0.00 -> 59.7 mm
- net PB11: track 0.00 -> 59.5 mm, vias 0 -> 1
- net /SD_MISO: track 0.00 -> 57.2 mm
- net PB10: track 0.00 -> 56.8 mm, vias 0 -> 1
- net /SD_MOSI: track 0.00 -> 56.3 mm
- net PE15: track 0.00 -> 54.1 mm, vias 0 -> 1
- net PA0: track 0.00 -> 52.0 mm
- net PB2: track 0.00 -> 51.8 mm, vias 0 -> 1
- net PA1: track 0.00 -> 51.5 mm
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- added copper zone on F.Cu, net GND
- added copper zone on In1.Cu, net GND
- added copper zone on F.Cu, net Net-(TP6-Pad1)
- added copper zone on F.Cu, net Net-(U1-VSS)
- added copper zone on In2.Cu, net Net-(U1-VSS)

Commit message: Another Update! :D
Parts:
- removed J6: 6130XX243121_613064243121, BQ25170DSGR:613064243121
- R7, TP37: moved to B.Cu
- moved TP37 185.3 mm to (28.5, 39.7)
- moved TP15 157.6 mm to (62.0, 99.7)
- moved R38 148.8 mm to (52.5, 41.6), turned to 90 degrees
- moved R31 145.5 mm to (53.0, 36.7), turned to -90 degrees
- moved R35 145.5 mm to (54.5, 39.7), turned to -90 degrees
- moved R28 145.4 mm to (46.0, 33.2), turned to 0 degrees
- moved R37 144.7 mm to (56.5, 39.7), turned to 90 degrees
- moved R36 143.6 mm to (58.0, 36.2), turned to -90 degrees
- moved R2 130.4 mm to (51.0, 36.2), turned to -90 degrees
- moved C1 123.0 mm to (49.0, 36.2), turned to -90 degrees
- moved R1 120.5 mm to (60.0, 34.7), turned to -90 degrees
- moved R7 111.4 mm to (27.5, 111.4), turned to -90 degrees
- moved TP11 105.0 mm to (106.5, 99.7)
- moved U6 100.6 mm to (55.1, 34.0)
- moved TP10 82.3 mm to (143.0, 116.7)
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Connections:
- U5 pad 100: PA11 -> unconnected-(U5B-PA11-Pad100)
- U5 pad 101: PA12 -> unconnected-(U5B-PA12-Pad101)
- U5 pad 131: PB4 -> unconnected-(U5B-PB4-Pad131)
- U5 pad 132: PB5 -> unconnected-(U5B-PB5-Pad132)
- U5 pad 133: PB6 -> unconnected-(U5B-PB6-Pad133)
- U5 pad 134: PB7 -> unconnected-(U5B-PB7-Pad134)
- U5 pad 136: PB8 -> unconnected-(U5B-PB8-Pad136)
- U5 pad 137: PB9 -> unconnected-(U5B-PB9-Pad137)
- U5 pad 138: PE0 -> unconnected-(U5B-PE0-Pad138)
- U5 pad 139: PE1 -> unconnected-(U5B-PE1-Pad139)
- U5 pad 2: PE3 -> unconnected-(U5A-PE3-Pad2)
- U5 pad 20: PF6 -> unconnected-(U5A-PF6-Pad20)
- U5 pad 21: PF7 -> unconnected-(U5A-PF7-Pad21)
- U5 pad 22: PF8 -> unconnected-(U5A-PF8-Pad22)
- U5 pad 23: PF9 -> unconnected-(U5A-PF9-Pad23)
- U5 pad 24: PF10 -> unconnected-(U5A-PF10-Pad24)
- U5 pad 28: PC0 -> unconnected-(U5A-PC0-Pad28)
- U5 pad 29: PC1 -> unconnected-(U5A-PC1-Pad29)
- U5 pad 3: PE4 -> unconnected-(U5A-PE4-Pad3)
- U5 pad 30: PC2_C -> unconnected-(U5A-PC2_C-Pad30)
- U5 pad 31: PC3_C -> unconnected-(U5A-PC3_C-Pad31)
- U5 pad 4: PE5 -> unconnected-(U5A-PE5-Pad4)
- U5 pad 5: PE6 -> unconnected-(U5A-PE6-Pad5)
- U5 pad 51: PB2 -> unconnected-(U5A-PB2-Pad51)
- U5 pad 52: PF11 -> unconnected-(U5A-PF11-Pad52)
- U5 pad 53: PF14 -> unconnected-(U5A-PF14-Pad53)
- U5 pad 54: PF15 -> unconnected-(U5A-PF15-Pad54)
- U5 pad 57: PE7 -> unconnected-(U5A-PE7-Pad57)
- U5 pad 58: PE8 -> unconnected-(U5A-PE8-Pad58)
- U5 pad 59: PE9 -> unconnected-(U5A-PE9-Pad59)
- U5 pad 60: PE10 -> unconnected-(U5A-PE10-Pad60)
- U5 pad 61: PE11 -> unconnected-(U5A-PE11-Pad61)
- U5 pad 62: PE12 -> unconnected-(U5A-PE12-Pad62)
- U5 pad 63: PE13 -> unconnected-(U5A-PE13-Pad63)
- U5 pad 64: PE14 -> unconnected-(U5A-PE14-Pad64)
- U5 pad 65: PE15 -> unconnected-(U5A-PE15-Pad65)
- U5 pad 66: PB10 -> unconnected-(U5A-PB10-Pad66)
- U5 pad 67: PB11 -> unconnected-(U5A-PB11-Pad67)
- U5 pad 77: PD9 -> unconnected-(U5B-PD9-Pad77)
- U5 pad 78: PD10 -> unconnected-(U5B-PD10-Pad78)
- U5 pad 81: PD11 -> unconnected-(U5B-PD11-Pad81)
- U5 pad 82: PD12 -> unconnected-(U5B-PD12-Pad82)
- U5 pad 83: PD13 -> unconnected-(U5B-PD13-Pad83)
- U5 pad 84: PD14 -> unconnected-(U5B-PD14-Pad84)
- U5 pad 85: PD15 -> unconnected-(U5B-PD15-Pad85)
- U5 pad 86: PG6 -> unconnected-(U5B-PG6-Pad86)
- U5 pad 87: PG7 -> unconnected-(U5B-PG7-Pad87)
- U5 pad 88: PG8 -> unconnected-(U5B-PG8-Pad88)
- U5 pad 93: PC6 -> unconnected-(U5B-PC6-Pad93)
- U5 pad 94: PC7 -> unconnected-(U5B-PC7-Pad94)
- U5 pad 95: PC8 -> unconnected-(U5B-PC8-Pad95)
- U5 pad 96: PC9 -> unconnected-(U5B-PC9-Pad96)
- U5 pad 97: PA8 -> unconnected-(U5B-PA8-Pad97)
- U5 pad 98: PA9 -> unconnected-(U5B-PA9-Pad98)
- U5 pad 99: PA10 -> unconnected-(U5B-PA10-Pad99)
Routing:
- net PB11: track 59.5 -> 0.00 mm, vias 1 -> 0
- net /Battery/PG: track 0.00 -> 57.5 mm
- net PB10: track 56.8 -> 0.00 mm, vias 1 -> 0
- net PE15: track 54.1 -> 0.00 mm, vias 1 -> 0
- net PA0: track 52.0 -> 0.00 mm
- net PB2: track 51.8 -> 0.00 mm, vias 1 -> 0
- net PA1: track 51.5 -> 0.00 mm
- net PE14: track 51.5 -> 0.00 mm, vias 1 -> 0
- net PE13: track 49.5 -> 0.00 mm, vias 1 -> 0
- net PF14: track 48.7 -> 0.00 mm, vias 1 -> 0
- net PE12: track 48.5 -> 0.00 mm, vias 1 -> 0
- net PE3: track 48.2 -> 0.00 mm
- net PF15: track 48.0 -> 0.00 mm, vias 1 -> 0
- net PE11: track 46.8 -> 0.00 mm, vias 1 -> 0
- net PE4: track 46.0 -> 0.00 mm
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
Commit message: pdf docs
Parts:
- moved TP1 145.5 mm to (23.0, 27.2)
- moved TP27 144.3 mm to (22.0, 30.7)
- moved TP13 125.6 mm to (24.5, 86.7)
- moved TP7 117.0 mm to (20.0, 111.4)
- moved TP3 112.2 mm to (65.0, 33.2)
- moved TP9 109.9 mm to (32.5, 93.7)
- moved TP5 108.2 mm to (54.5, 43.7)
- moved TP2 66.5 mm to (194.0, 67.2)
- moved C8 65.1 mm to (106.5, 88.7), turned to 0 degrees
- moved TP4 64.1 mm to (92.0, 63.7)
- moved TP36 63.2 mm to (191.5, 63.2)
- moved R25 59.6 mm to (111.5, 85.2), turned to 180 degrees
- moved R24 57.7 mm to (112.0, 92.7), turned to 180 degrees
- moved J7 47.4 mm to (148.5, 74.2)
- moved TP8 43.2 mm to (160.0, 80.2)
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
Commit message: PCB about 75% done
Parts:
- R10, R11, R12, R15, R16, R17, R7, R9: moved to F.Cu
- moved TP36 161.8 mm to (32.5, 33.2), turned to 180 degrees
- moved TP2 156.7 mm to (41.0, 33.2), turned to 180 degrees
- moved R27 155.0 mm to (39.4, 36.7), turned to -90 degrees
- moved R29 151.3 mm to (42.4, 36.7), turned to -90 degrees
- moved CR1 149.7 mm to (39.4, 41.2), turned to -90 degrees
- moved CR2 145.8 mm to (42.5, 41.2), turned to -90 degrees
- moved R18 145.0 mm to (24.0, 83.2), turned to -90 degrees
- moved C4 140.2 mm to (43.0, 47.7)
- moved C5 134.2 mm to (46.5, 45.2), turned to 90 degrees
- moved TP14 133.8 mm to (52.0, 100.5), turned to -90 degrees
- moved U4 132.2 mm to (47.0, 48.5), turned to 180 degrees
- moved R6 131.7 mm to (48.5, 42.2), turned to 90 degrees
- moved R5 130.3 mm to (48.5, 45.2), turned to 90 degrees
- moved R8 126.6 mm to (40.0, 111.2), turned to -90 degrees
- moved TP8 124.7 mm to (40.0, 114.2)
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Connections:
- D2 pad 1: unconnected-(D2-K-Pad1) -> GND
- U4 pad V: (no net) -> GND
- U6 pad 10: (no net) -> GND
Routing:
- net +3.3V: track 0.00 -> 343.3 mm, vias 0 -> 12
- net /Controllers/SlideSwitch: track 0.00 -> 74.4 mm, vias 0 -> 2
- net /SWO: track 0.00 -> 66.7 mm, vias 0 -> 2
- net /Battery/BAT_DIAG: track 0.00 -> 64.7 mm, vias 0 -> 2
- net /nRESET: track 0.00 -> 55.3 mm, vias 0 -> 2
- net /Battery/PACK+: track 0.00 -> 51.1 mm, vias 0 -> 7
- net /SWCLK: track 0.00 -> 48.4 mm
- net /SWDIO: track 0.00 -> 46.2 mm
- net Net-(R34-Pad2): track 0.00 -> 33.0 mm, vias 0 -> 2
- net Net-(U5A-PE2): track 0.00 -> 30.9 mm, vias 0 -> 2
- net Net-(U1-VSS): track 0.00 -> 22.9 mm, vias 18 -> 11
- net GND: track 7.78 -> 29.9 mm, vias 33 -> 63
- net Net-(R33-Pad1): track 0.00 -> 21.2 mm
- net Net-(J5-Pad3): track 0.00 -> 14.3 mm
- net Net-(C5-Pad1): track 0.00 -> 12.3 mm
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- added copper zone on B.Cu, net /Battery/PACK+
- added copper zone on F.Cu, net /Battery/PACK+
- added copper zone on B.Cu, net Net-(U1-VSS)
- added copper zone on F.Cu, net Net-(U4-AVIN)
- removed copper zone on In2.Cu, net Net-(U1-VSS)
